File: My Projects.kicad_sch (KiCad schematic)
At the start: 12 parts, among them IC1 7483, IC2 7483, IC3 7486, IC4 7486, SW1 SW_SPST, SW2 SW_SPST, SW3 SW_SPST, SW4 SW_SPST, SW5 SW_SPST, SW6 SW_SPST, SW7 SW_SPST, SW8 SW_SPST

Commit message: COMMIT
Parts:
- added D1, D2, D3, D4, D5, D6, D7, D8: LED, symbol Device:LED
- added R1, R2, R3, R4, R5, R6, R7, R8: R, symbol Device:R
Connections:
- net B0: now also D8.2 (A)
- net B1: now also D7.2 (A)
- net B2: now also D6.2 (A)
- net B3: now also D5.2 (A)
- net B4: now also D4.2 (A)
- net B5: now also D3.2 (A)
- net B6: now also D2.2 (A)
- net B7: now also D1.2 (A)
- net at SW1.1 (A): now also R1.1
- net at SW6.1 (A): now also R6.1
- net at SW7.1 (A): now also R7.1
- net at SW5.1 (A): now also R5.1
- net at SW2.1 (A): now also R2.1
- net SUB: now reaches IC2.13 (C0), IC3.10, IC3.13, IC3.2, IC3.5, IC4.10, IC4.13, IC4.2, IC4.5
- net at SW3.1 (A): now also R3.1
- net at SW4.1 (A): now also R4.1
- net at SW8.1 (A): now also R8.1
- new net: D4.1 (K), R4.2
- new net: D8.1 (K), R8.2
- new net: D7.1 (K), R7.2
- new net: D2.1 (K), R2.2
- new net: D5.1 (K), R5.2
- new net: D3.1 (K), R3.2
- new net: D6.1 (K), R6.2
- new net: D1.1 (K), R1.2

Commit message: COMMIT
Parts:
- added D10, D11, D12, D13, D14, D15, D16, D9: LED, symbol Device:LED
- added R10, R11, R12, R13, R14, R15, R16, R9: R, symbol Device:R
Connections:
- net S7: now reaches IC1.15 (S3)
- net S7: now also R9.1
- net S6: now reaches IC1.2 (S2)
- net S6: now also R10.1
- net S5: now reaches IC1.6 (S1)
- net S5: now also R11.1
- net S4: now reaches IC1.9 (S0)
- net S4: now also R12.1
- net S3: now reaches IC2.15 (S3)
- net S3: now also R13.1
- net S2: now reaches IC2.2 (S2)
- net S2: now also R14.1
- net S1: now reaches IC2.6 (S1)
- net S1: now also R15.1
- net S0: now reaches IC2.9 (S0)
- net S0: now also R16.1
- new net: D14.2 (A), R14.2
- new net: D13.2 (A), R13.2
- new net: D16.2 (A), R16.2
- new net: D12.2 (A), R12.2
- new net: D15.2 (A), R15.2
- new net: D10.2 (A), R10.2
- new net: D11.2 (A), R11.2
- new net: D9.2 (A), R9.2

Commit message: COMMIT
Connections:
- net GND: now also SW1.2 (B), SW2.2 (B), SW3.2 (B), SW4.2 (B), SW5.2 (B), SW6.2 (B), SW7.2 (B), SW8.2 (B)
Changed lines of the file:
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@@
+	)
+	(junction
+		(at 104.14 17.78)
+		(diameter 0)
+		(color 0 0 0 0)
+	)
+	(junction
+		(at 201.93 17.78)
+		(diameter 0)
+		(color 0 0 0 0)
 	)
 	(junction
@@
 	)
 	(junction
+		(at 123.19 17.78)
+		(diameter 0)
+		(color 0 0 0 0)
+	)
+	(junction
+		(at 189.23 17.78)
+		(diameter 0)
+		(color 0 0 0 0)
+	)
+	(junction
 		(at 125.73 49.53)
 		(diameter 0)
@@
 	)
 	(junction
+		(at 116.84 17.78)
+		(diameter 0)
+		(color 0 0 0 0)
+	)
+	(junction
+		(at 59.69 128.27)
+		(diameter 0)
+		(color 0 0 0 0)
+	)
+	(junction
+		(at 194.31 17.78)
+		(diameter 0)
+		(color 0 0 0 0)
+	)
+	(junction
 		(at 119.38 49.53)
 		(diameter 0)
 		(color 0 0 0 0)
 	)
+	(junction
+		(at 109.22 17.78)
+		(diameter 0)
+		(color 0 0 0 0)
+	)
 	(no_connect
 		(at 69.85 120.65)
@@
 	(wire
 		(pts
+			(xy 194.31 17.78) (xy 201.93 17.78)
+		)
+		(stroke
+			(width 0)
+			(type default)
+		)
+	)
+	(wire
+		(pts
 			(xy 198.12 49.53) (xy 204.47 49.53)
 		)
@@
 	(wire
 		(pts
+			(xy 116.84 17.78) (xy 123.19 17.78)
+		)
+		(stroke
+			(width 0)
+			(type default)
+		)
+	)
+	(wire
+		(pts
 			(xy 125.73 49.53) (xy 191.77 49.53)
 		)
@@
 	(wire
 		(pts
+			(xy 104.14 17.78) (xy 109.22 17.78)
+		)
+		(stroke
+			(width 0)
+			(type default)
+		)
+	)
+	(wire
+		(pts
 			(xy 125.73 49.53) (xy 125.73 64.77)
 		)
@@
 	(wire
 		(pts
+			(xy 45.72 128.27) (xy 59.69 128.27)
+		)
+		(stroke
+			(width 0)
+			(type default)
+		)
+	)
+	(wire
+		(pts
 			(xy 191.77 49.53) (xy 198.12 49.53)
 		)
@@
 	(wire
 		(pts
+			(xy 45.72 17.78) (xy 45.72 128.27)
+		)
+		(stroke
+			(width 0)
+			(type default)
+		)
+	)
+	(wire
+		(pts
 			(xy 106.68 49.53) (xy 113.03 49.53)
 		)
@@
 	(wire
 		(pts
+			(xy 104.14 17.78) (xy 45.72 17.78)
+		)
+		(stroke
+			(width 0)
+			(type default)
+		)
+	)
+	(wire
+		(pts
 			(xy 210.82 49.53) (xy 210.82 60.96)
 		)
@@
 	(wire
 		(pts
+			(xy 189.23 17.78) (xy 194.31 17.78)
+		)
+		(stroke
+			(width 0)
+			(type default)
+		)
+	)
+	(wire
+		(pts
 			(xy 123.19 58.42) (xy 123.19 64.77)
 		)
@@
 	(wire
 		(pts
+			(xy 201.93 17.78) (xy 208.28 17.78)
+		)
+		(stroke
+			(width 0)
+			(type default)
+		)
+	)
+	(wire
+		(pts
+			(xy 59.69 128.27) (xy 72.39 128.27)
+		)
+		(stroke
+			(width 0)
+			(type default)
+		)
+	)
+	(wire
+		(pts
+			(xy 59.69 128.27) (xy 59.69 129.54)
+		)
+		(stroke
+			(width 0)
+			(type default)
+		)
+	)
+	(wire
+		(pts
 			(xy 201.93 83.82) (xy 201.93 97.79)
 		)
@@
 	(wire
 		(pts
+			(xy 109.22 17.78) (xy 116.84 17.78)
+		)
+		(stroke
+			(width 0)
+			(type default)
+		)
+	)
+	(wire
+		(pts
 			(xy 189.23 55.88) (xy 189.23 60.96)
 		)
@@
 		(pts
 			(xy 116.84 58.42) (xy 116.84 64.77)
+		)
+		(stroke
+			(width 0)
+			(type default)
+		)
+	)
+	(wire
+		(pts
+			(xy 123.19 17.78) (xy 189.23 17.78)
 		)
 		(stroke
@@
 	(symbol
 		(lib_id "power:GND")
-		(at 72.39 128.27 0)
+		(at 59.69 129.54 0)
 		(unit 1)
 		(exclude_from_sim no)
@@
 		(fields_autoplaced yes)
 		(property "Reference" "#PWR03"
-			(at 72.39 134.62 0)
+			(at 59.69 135.89 0)
 			(effects
 				(font
@@
 		)
 		(property "Value" "GND"
-			(at 72.39 133.35 0)
+			(at 59.69 134.62 0)
 			(effects
 				(font
@@
 		)
 		(property "Footprint" ""
-			(at 72.39 128.27 0)
+			(at 59.69 129.54 0)
 			(effects
 				(font
@@
 		)
 		(property "Datasheet" ""
-			(at 72.39 128.27 0)
+			(at 59.69 129.54 0)
 			(effects
 				(font
@@
 		)
 		(property "Description" "Power symbol creates a global label with name \"GND\" , ground"
-			(at 72.39 128.27 0)
-			(effects
-				(font
+			(at 59.69 129.54 0)
+			(effects
+				(font
